Commit message: new stuff added for trajectory_planning

File: umirtx_description/urdf/UMI_RTX_URDF.urdf (robot description, URDF)
Before this commit: robot UMI_RTX_BM14W4, 11 links, 10 joints
Links:
- link base_link: mass 100 -> None
- link frametip: geometry collision box size=0.11 0.021 0.11; visual box size=0.1 0.02 0.10
Joints:
- joint jointtip: origin xyz=0.130 0.0 0.035 rpy=0 0 0 -> xyz=0.0 0.00 0.08 rpy=0 0 0
